File: Board/Remote/remote.brd (EAGLE design)
At the start: 81.9 x 39.4 mm, 32 parts, among them U2 ATMEGA328P_TQFP, Y1 16MHz

Commit message: Latest board layout - what was sent to oshpark.
Parts:
- removed S1: SWITCH-MOMENTARY-2PTH, SparkFun-Electromechanical:TACTILE-PTH
- added C3, C5: 10UF, adafruit:A/3216-18W
- added C4: 1UF, adafruit:C0805
- added IC1: MCP1253-33X50, microchip-MCP125x-xxx:MSOP8
- added R10: 100k, adafruit:R0805
- added R11, R12: 4K7, adafruit:R0805
- C1, C2: device SparkFun-Capacitors:CAP-PTH-SMALL -> adafruit:C0805
- JP3: value M09 -> (none); device SparkFun-Connectors:1X09 -> SparkFun-Connectors:1X06
- moved LED2 50.7 mm to (73.7, 27.3)
- moved R8 44.7 mm to (71.1, 27.3), turned to 270 degrees
- moved R9 43.3 mm to (68.6, 27.3)
- moved LED1 42.1 mm to (66.0, 27.3)
- moved R1 22.5 mm to (48.3, 27.9), turned to 90 degrees
- moved U$1 13.6 mm to (65.4, 10.8), turned to 90 degrees
- moved R2 9.44 mm to (68.6, 19.7), turned to 90 degrees
- moved IRSENSOR 5.08 mm to (5.08, 22.9), turned to 90 degrees
- moved JP3 3.17 mm to (50.2, 37.5)
- moved R7 1.42 mm to (80.6, 12.7)
- moved R5 1.27 mm to (38.1, 15.2)
- moved R6 1.27 mm to (14.0, 15.2)
- moved C1 1.27 mm to (48.3, 17.8)
- moved C2 1.27 mm to (64.8, 17.8), turned to 90 degrees
- moved R3 1.27 mm to (38.1, 24.1)
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Connections:
- removed net VCC: IRSENSOR.1, JP4.2, POWER.2, R1.2, S2.3, S3.3, S4.3, S5.3, S6.3, U$1.8, U2.18, U2.20, U2.4, U2.6
- new net 5V: C3.+, IC1.2, IRSENSOR.1, JP4.2, R1.2, R10.1, R11.1, R12.1, S2.3, S3.3, S4.3, S5.3, S6.3, U$1.8, U2.18, U2.20, U2.4, U2.6
- new net N$7: C4.1, IC1.5
- new net N$8: C4.2, IC1.6
- new net VBAT: C5.+, IC1.3, IC1.7, POWER.2
- net B0: now also JP3.4; no longer JP3.5
- net B1: now also JP3.5; no longer JP3.6
- net B2: now also JP3.6; no longer JP3.7
- net B4/MISO: no longer JP3.8
- net B5/SCK: no longer JP3.9
- net D4: now also IC1.1, R10.2; no longer JP3.3
- net D5: now also JP3.3; no longer JP3.4
- net GND: now also C2.1, C3.-, C5.-, IC1.4, IC1.8; no longer C2.2, S1.1
- net N$3: now also C2.2; no longer C2.1
- net RESET: no longer S1.3
- net SCL: now also R12.2
- net SDA: now also R11.2
Routing:
- net 5V: track 0.00 -> 273.7 mm, vias 0 -> 2
- net VCC: track 209.9 -> 0.00 mm, vias 2 -> 0
- net D4: track 21.4 -> 67.1 mm, vias 0 -> 2
- net D7: track 40.7 -> 8.53 mm, vias 2 -> 0
- net RESET: track 65.4 -> 34.8 mm, vias 2 -> 0
- net VBAT: track 0.00 -> 30.1 mm
- net D6: track 41.1 -> 11.0 mm, vias 2 -> 0
- net C2: track 82.0 -> 55.0 mm, vias 2 -> 0
- net D2: track 49.4 -> 70.0 mm
- net SDA: track 30.3 -> 44.0 mm, vias 1 -> 0
- net D3: track 46.3 -> 34.1 mm
- net GND: track 72.0 -> 83.7 mm, vias 2 -> 8
- net B5/SCK: track 51.8 -> 40.1 mm, vias 1 -> 0
- net B0: track 20.2 -> 12.5 mm
- net SCL: track 42.3 -> 36.3 mm, vias 0 -> 2
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Other:
- outline, holes or cut-outs redrawn
- board text added: "BAT"
- board text added: "NC"
- board text added: "Remote v1"
