File: Board/Remote/remote.sch (EAGLE design)
At the start: 32 parts, among them U2 ATMEGA328P_TQFP, Y1 16MHz

Commit message: Latest board layout - what was sent to oshpark.
Parts:
- removed S1: SWITCH-MOMENTARY-2PTH, SparkFun-Electromechanical:SWITCH-MOMENTARY-2PTH
- added C3, C5: 10UF, adafruit:CPOL-USA/3216-18W
- added C4: 1UF, adafruit:C-USC0805
- added IC1: MCP1253-33X50, microchip-MCP125x-xxx:MCP1253-33X50
- added R10: 100k, adafruit:R-US_R0805
- added R11, R12: 4K7, adafruit:R-US_R0805
- C1, C2: device SparkFun-Capacitors:CAPPTH -> adafruit:C-USC0805
- JP3: value M09 -> (none); device SparkFun-Connectors:M09 -> SparkFun-Connectors:M06SIP
Connections:
- removed net VCC: IRSENSOR.1, JP4.2, POWER.2, R1.2, S2.2, S3.2, S4.2, S5.2, S6.2, U$1.VCC, U2.AREF, U2.AVCC, U2.VCC@4, U2.VCC@6
- new net 5V: C3.+, IC1.VOUT, IRSENSOR.1, JP4.2, R1.2, R10.1, R11.1, R12.1, S2.2, S3.2, S4.2, S5.2, S6.2, U$1.VCC, U2.AREF, U2.AVCC, U2.VCC@4, U2.VCC@6
- new net N$7: C4.1, IC1.C-
- new net N$8: C4.2, IC1.C+
- new net VBAT: C5.+, IC1.SHDN, IC1.VIN, POWER.2
- net B0: now also JP3.4; no longer JP3.5
- net B1: now also JP3.5; no longer JP3.6
- net B2: now also JP3.6; no longer JP3.7
- net B4/MISO: no longer JP3.8
- net B5/SCK: no longer JP3.9
- net D4: now also IC1.PGOOD, R10.2; no longer JP3.3
- net D5: now also JP3.3; no longer JP3.4
- net GND: now also C2.1, C3.-, C5.-, IC1.GND, IC1.SELECT; no longer C2.2, S1.1
- net N$3: now also C2.2; no longer C2.1
- net RESET: no longer S1.2
- net SCL: now also R12.2
- net SDA: now also R11.2
Other:
- moved on the sheet: C1, C2
